File: MiniRC.kicad_sch (KiCad schematic)
At the start: 45 parts, among them J2 Conn_02x04_Odd_Even, J3 Conn_01x04_Socket, J4 Conn_02x08_Odd_Even, J5 Conn_01x04_Pin, J6 Conn_01x02_Pin, J7 Conn_01x02_Pin, J8 Conn_01x02_Pin, SW1 SW_Push, U1 STM32F103C8Tx, U5 TB6612FNG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

Commit message: Organise details
Parts:
- C14, C16, C17: value 0.1uF -> 100nF
Changed lines of the file:
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@@
 			)
 		)
-		(property "Value" "0.1uF"
+		(property "Value" "100nF"
 			(at 181.61 60.198 90)
 			(effects
@@
 			)
 		)
-		(property "Value" "0.1uF"
+		(property "Value" "100nF"
 			(at 152.4 26.67 90)
 			(effects
@@
 			)
 		)
-		(property "Value" "0.1uF"
+		(property "Value" "100nF"
 			(at 173.99 25.908 90)
 			(effects

Commit message: Organise details
Connections:
- net +5V: no longer C28.1, C29.1, C8.1, U5.13 (VM2), U5.14 (VM3), U5.24 (VM1)
- net BAT_OUT: now also C28.1, C29.1, C8.1, U5.13 (VM2), U5.14 (VM3), U5.24 (VM1)
Changed lines of the file:
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@@
-	)
-	(junction
-		(at 143.51 87.63)
-		(diameter 0)
-		(color 0 0 0 0)
 	)
 	(junction
@@
 	(wire
 		(pts
-			(xy 143.51 87.63) (xy 153.67 87.63)
-		)
-		(stroke
-			(width 0)
-			(type default)
-		)
-	)
-	(wire
-		(pts
 			(xy 27.94 168.91) (xy 27.94 167.64)
 		)
@@
 		(pts
 			(xy 247.65 19.05) (xy 259.08 19.05)
+		)
+		(stroke
+			(width 0)
+			(type default)
+		)
+	)
+	(wire
+		(pts
+			(xy 149.86 87.63) (xy 153.67 87.63)
 		)
 		(stroke
@@
 		)
 	)
+	(label "BAT_OUT"
+		(at 149.86 87.63 90)
+		(effects
+			(font
+				(size 1.27 1.27)
+			)
+			(justify left bottom)
+		)
+	)
