File: power.kicad_sch (KiCad schematic)
At the start: 28 parts, among them J1 Conn_01x02_Pin, U3 AMS1117-3.3, U4 MT3608, U8 AMS1117-3.3, U9 TPS54302

Commit message: Organise details
Parts:
- C23, C24: value 0.1uF -> 100nF
- C27: value 75pF -> 100pF
- R13: value 100k -> 82k
- R14: value 13.3k -> 11k
Changed lines of the file:
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@@
 			)
 		)
-		(property "Value" "0.1uF"
+		(property "Value" "100nF"
 			(at 91.694 34.29 0)
 			(effects
@@
 			)
 		)
-		(property "Value" "75pF"
+		(property "Value" "100pF"
 			(at 157.734 44.45 0)
 			(effects
@@
 			)
 		)
-		(property "Value" "100k"
+		(property "Value" "82k"
 			(at 172.72 44.4499 0)
 			(effects
@@
 			)
 		)
-		(property "Value" "0.1uF"
+		(property "Value" "100nF"
 			(at 134.62 20.32 90)
 			(effects
@@
 			)
 		)
-		(property "Value" "13.3k"
+		(property "Value" "11k"
 			(at 172.72 54.6099 0)
 			(effects

Commit message: Organise details
Parts:
- added TP1: B-, TestPoint:TestPoint_Pad_D2.0mm, symbol Connector:TestPoint
- added TP2: VIN, TestPoint:TestPoint_Pad_D2.0mm, symbol Connector:TestPoint
- added TP3: B+, TestPoint:TestPoint_Pad_D2.0mm, symbol Connector:TestPoint
- added TP4: GND, TestPoint:TestPoint_Pad_D2.0mm, symbol Connector:TestPoint
- D2, D3: footprint Diode_SMD:D_SMA -> Diode_SMD:D_SMC_Handsoldering
Connections:
- net GND: now also TP1.1
- net VBAT_RAW: now reaches D2.1 (K), J1.2 (Pin_2)
- net VBAT_RAW: now also TP3.1
- no-connect marks 0 -> 2
