File: MiniRC.kicad_pcb (KiCad board)
At the start: 2 copper layers, 113.5 x 63.9 mm, 89 parts, among them J1 Conn_01x02_Pin, J2 Conn_02x04_Odd_Even, J3 Conn_01x04_Socket, J4 Conn_02x08_Odd_Even, J5 Conn_01x04_Pin, J6 Conn_01x02_Pin, J7 Conn_01x02_Pin, J8 Conn_01x02_Pin, J9 Conn_01x02_Pin, Q1 NMOS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

Commit message: Organise details
Parts:
- removed the G*** at (232.5, 31.6)
- added G***: LOGO, icons:eye, B.Cu at (139.7, 34.0)
- C11: footprint Capacitor_SMD:C_1206_3216Metric_Pad1.33x1.80mm_HandSolder -> Capacitor_THT:C_Disc_D10.5mm_W5.0mm_P10.00mm
- C14, C16, C17, C23, C24: value 0.1uF -> 100nF
- moved C11 0.33 mm to (142.1, 51.4), turned to -90 degrees
Routing:
- net Net-(J9-Pin_2): track 10.3 -> 15.0 mm
- net Net-(C11-Pad1): track 2.92 -> 4.90 mm
- net GND: vias 193 -> 189

Commit message: Organise details
Parts:
- removed the REF** at (128.8, 85.5)
- added TP1: B-, TestPoint:TestPoint_Pad_D2.0mm, B.Cu at (128.6, 56.4)
- added TP2: VIN, TestPoint:TestPoint_Pad_D2.0mm, B.Cu at (128.6, 86.4)
- added TP3: B+, TestPoint:TestPoint_Pad_D2.0mm, B.Cu at (146.6, 56.4)
- added TP4: GND, TestPoint:TestPoint_Pad_D2.0mm, B.Cu at (146.6, 86.4)
- C27: value 75pF -> 100pF
- D2, D3: footprint Diode_SMD:D_SMA -> Diode_SMD:D_SMC_Handsoldering
- D4, D5: footprint Diode_SMD:D_0805_2012Metric_Pad1.15x1.40mm_HandSolder -> Diode_SMD:D_SMA_Handsoldering
- R13: value 100k -> 82k
- R14: value 13.3k -> 11k
- moved J9 5.50 mm to (131.2, 39.9)
- moved C7 4.71 mm to (170.7, 69.2), turned to 0 degrees
- moved D5 3.50 mm to (143.2, 45.2)
- moved D3 3.45 mm to (175.5, 74.0)
- moved D4 3.40 mm to (143.3, 41.4)
- moved D2 3.19 mm to (141.2, 70.2)
- moved C8 1.71 mm to (184.3, 76.8)
- moved C29 1.12 mm to (184.6, 72.3)
- moved J1 0.80 mm to (130.7, 61.8)
Connections:
- net Net-(D2-K) renamed VBAT_RAW
- C28 pad 1: +5V -> /BAT_OUT
- C29 pad 1: +5V -> /BAT_OUT
- C8 pad 1: +5V -> /BAT_OUT
- U5 pad 13: +5V -> /BAT_OUT
- U5 pad 14: +5V -> /BAT_OUT
- U5 pad 24: +5V -> /BAT_OUT
Routing:
- net /BAT_OUT: track 55.4 -> 106.1 mm, vias 0 -> 2
- net +5V: track 152.8 -> 131.9 mm
- net VBAT_RAW: track 5.45 -> 23.7 mm, vias 0 -> 1
- net GND: track 33.1 -> 45.3 mm, vias 189 -> 181
- net Net-(D3-A): track 28.1 -> 24.4 mm
- net Net-(J9-Pin_2): track 15.0 -> 18.2 mm
- net Net-(J8-Pin_2): track 22.3 -> 23.7 mm
- net Net-(J8-Pin_1): track 18.3 -> 19.6 mm
- net +24V: track 48.3 -> 49.4 mm
- net Net-(D4-A): track 27.4 -> 26.7 mm
Other:
- board text added: "CHARGER"

Commit message: Organise details
Parts:
- removed the G*** at (139.7, 34.0)
- moved G*** 3.10 mm to (139.5, 31.6)
- moved J2 1.98 mm to (215.0, 81.0)
Routing:
- net SPI1_SCK: track 27.8 -> 30.0 mm
- net RF_IRQ: track 18.6 -> 20.7 mm
- net SPI1_MOSI: track 21.4 -> 23.3 mm
- net CE: track 30.1 -> 31.9 mm
- net CSN: track 24.6 -> 26.2 mm
- net /+3.3V_RADIO: track 49.8 -> 51.4 mm
- net GND: track 45.3 -> 44.1 mm, vias 181 -> 180
- net Net-(J8-Pin_2): track 23.7 -> 23.0 mm
- net +5V: vias 4 -> 3
Other:
- board size 113.5 x 63.9 mm -> 113.5 x 64 mm

Commit message: Update
Parts:
- added REF**: MountingHole_2.1mm, MountingHole:MountingHole_2.1mm, F.Cu at (165.0, 86.3)
- moved TP1 3.40 mm to (132.0, 56.4)
- moved TP2 3.40 mm to (132.0, 86.4)
- moved TP3 3.40 mm to (150.0, 56.4)
- moved TP4 3.40 mm to (150.0, 86.4)
Routing:
- net VBAT_RAW: track 23.7 -> 29.3 mm
- net /BAT_OUT: track 106.1 -> 106.9 mm
- net GND: track 44.1 -> 44.8 mm, vias 180 -> 177
